Commit message: Add new files and make changes to existing files

File: python_scripts/urdf/quadbot.urdf (robot description, URDF)
Before this commit: robot quadbot, 6 links, 5 joints
Links:
- removed link FR_1_link
- removed link FR_2_link
- removed link FR_3_link
- removed link FR_4_link
- removed link FR_link
- added link fr_link_0, mass 0.0926222295025173; collision mesh filename=../meshes/fr_link_0.STL; visual mesh filename=../meshes/fr_link_0.STL
- link base_link: mass 1.1069 -> 0.996322261989855
Joints:
- removed joint FR_1_joint
- removed joint FR_2_joint
- removed joint FR_3_joint
- removed joint FR_4_joint
- removed joint FR_joint
- added joint fr_jnt_0: type revolute, parent base_link, child fr_link_0, origin xyz=0.20229 0.19155 0.095 rpy=-1.5708 -0.0068295 1.5708, axis 0 0 -1, limit lower=0 upper=0 effort=0 velocity=0
