Commit message: Update simulation loading script and URDF file for quadson robot

File: quadson-sim/urdf/quadson.urdf (robot description, URDF)
Before this commit: robot quadson, 21 links, 20 joints
Links:
- link base_link_.002_link: geometry collision mesh filename=../meshes/dae/base_link.004.dae scale=1.00000 1.00000 1.00000; visual mesh filename=../meshes/dae/base_link.004.dae scale=1.00000 1.00000 1.00000

Commit message: Enable collision object in simulation

File: quadson-sim/urdf/quadson.urdf (robot description, URDF)
Before this commit: robot quadson, 21 links, 20 joints
Links:
- removed link base_link_.002_link
- removed link fr_link0.002
- removed link fr_llink1.002
- removed link fr_llink2.002
- removed link fr_llink3.002
- removed link fr_llink4.002
- removed link link0.002
- removed link link0.003
- removed link link0.004
- removed link link1.002
- removed link link1.003
- removed link link1.004
- removed link link2.002
- removed link link2.003
- removed link link2.004
- removed link link3.002
- removed link link3.003
- removed link link3.004
- removed link link4.001
- removed link link4.004
- removed link link4.005
- added link base_link, mass 1.50000; visual mesh filename=../meshes/dae/base_link.dae scale=1.00000 1.00000 1.00000
- added link bl_link0, mass 0.40000; visual mesh filename=../meshes/dae/bl_link0.dae scale=1.00000 1.00000 1.00000
- added link bl_link1, mass 0.20000; visual mesh filename=../meshes/dae/bl_link1.dae scale=1.00000 1.00000 1.00000
- added link bl_link2, mass 0.20000; visual mesh filename=../meshes/dae/bl_link2.dae scale=1.00000 1.00000 1.00000
- added link bl_link3, mass 0.20000; visual mesh filename=../meshes/dae/bl_link3.dae scale=1.00000 1.00000 1.00000
- added link bl_link4, mass 0.20000; visual mesh filename=../meshes/dae/bl_link4.dae scale=1.00000 1.00000 1.00000
- added link br_link0, mass 0.40000; visual mesh filename=../meshes/dae/br_link0.dae scale=1.00000 1.00000 1.00000
- added link br_link1, mass 0.20000; visual mesh filename=../meshes/dae/br_link1.dae scale=1.00000 1.00000 1.00000
- added link br_link2, mass 0.20000; visual mesh filename=../meshes/dae/br_link2.dae scale=1.00000 1.00000 1.00000
- added link br_link3, mass 0.20000; visual mesh filename=../meshes/dae/br_link3.dae scale=1.00000 1.00000 1.00000
- added link br_link4, mass 0.20000; visual mesh filename=../meshes/dae/br_link4.dae scale=1.00000 1.00000 1.00000
- added link fl_link0, mass 0.40000; visual mesh filename=../meshes/dae/fl_link0.dae scale=1.00000 1.00000 1.00000
- added link fl_link1, mass 0.20000; visual mesh filename=../meshes/dae/fl_link1.dae scale=1.00000 1.00000 1.00000
- added link fl_link2, mass 0.20000; visual mesh filename=../meshes/dae/fl_link2.dae scale=1.00000 1.00000 1.00000
- added link fl_link3, mass 0.20000; visual mesh filename=../meshes/dae/fl_link3.dae scale=1.00000 1.00000 1.00000
- added link fl_link4, mass 0.20000; visual mesh filename=../meshes/dae/fl_link4.dae scale=1.00000 1.00000 1.00000
- added link fr_link0, mass 0.40000; visual mesh filename=../meshes/dae/fr_link0.dae scale=1.00000 1.00000 1.00000
- added link fr_link1, mass 0.20000; visual mesh filename=../meshes/dae/fr_link1.dae scale=1.00000 1.00000 1.00000
- added link fr_link2, mass 0.20000; visual mesh filename=../meshes/dae/fr_link2.dae scale=1.00000 1.00000 1.00000
- added link fr_link3, mass 0.20000; visual mesh filename=../meshes/dae/fr_link3.dae scale=1.00000 1.00000 1.00000
- added link fr_link4, mass 0.20000; visual mesh filename=../meshes/dae/fr_link4.dae scale=1.00000 1.00000 1.00000
Joints:
- removed joint fl_jjoint2
- removed joint fl_jjoint3
- removed joint fl_jjoint4
- added joint fl_joint2: type revolute, parent fl_link1, child fl_link2, origin xyz=0.04173 0.06842 0.00768 rpy=-0.00000 -0.00000 -0.00000, axis 0.00000 0.00000 1.00000, limit lower=-3.14000 upper=3.14000 effort=0.00000 velocity=0.00000
- added joint fl_joint3: type revolute, parent fl_link2, child fl_link3, origin xyz=-0.05988 0.08000 -0.00045 rpy=-0.00000 0.00000 -0.00000, axis 0.00000 0.00000 1.00000, limit lower=-3.14000 upper=3.14000 effort=0.00000 velocity=0.00000
- added joint fl_joint4: type revolute, parent fl_link3, child fl_link4, origin xyz=-0.10334 -0.07887 0.00054 rpy=-0.00000 -0.00000 0.00000, axis 0.00000 0.00000 1.00000, limit lower=-3.14000 upper=3.14000 effort=0.00000 velocity=0.00000
- joint bl_joint0: child link0.003 -> bl_link0; origin xyz=-0.20768 0.09541 0.00215 rpy=-0.00000 1.57080 0.00000 -> xyz=-0.20768 0.09541 0.00215 rpy=0.00000 1.57080 0.00000; parent base_link_.002_link -> base_link
- joint bl_joint1: child link1.003 -> bl_link1; parent link0.003 -> bl_link0
- joint bl_joint2: child link2.003 -> bl_link2; parent link1.003 -> bl_link1
- joint bl_joint3: child link3.003 -> bl_link3; parent link2.003 -> bl_link2
- joint bl_joint4: child link4.004 -> bl_link4; parent link3.003 -> bl_link3
- joint br_joint0: child link0.002 -> br_link0; origin xyz=-0.20768 -0.09459 0.00215 rpy=-0.00000 1.57080 0.00000 -> xyz=-0.20768 -0.09459 0.00215 rpy=0.00000 1.57080 0.00000; parent base_link_.002_link -> base_link
- joint br_joint1: child link1.002 -> br_link1; origin xyz=0.00040 -0.01862 0.05458 rpy=1.57080 -1.57080 0.00000 -> xyz=0.00040 -0.01862 0.05458 rpy=1.57080 -1.57080 -0.00000; parent link0.002 -> br_link0
- joint br_joint2: child link2.002 -> br_link2; parent link1.002 -> br_link1
- joint br_joint3: child link3.002 -> br_link3; parent link2.002 -> br_link2
- joint br_joint4: child link4.001 -> br_link4; parent link3.002 -> br_link3
- joint fl_jjoint1: child link1.004 -> fl_link1; origin xyz=-0.00040 0.01862 0.05430 rpy=-1.57080 1.57080 0.00000 -> xyz=-0.00040 0.01862 0.05430 rpy=-1.57080 1.57080 -0.00000; parent link0.004 -> fl_link0
- joint fl_joint0: child link0.004 -> fl_link0; parent base_link_.002_link -> base_link
- joint fr_joint0: child fr_link0.002 -> fr_link0; parent base_link_.002_link -> base_link
- joint fr_joint1: child fr_llink1.002 -> fr_link1; parent fr_link0.002 -> fr_link0
- joint fr_joint2: child fr_llink2.002 -> fr_link2; parent fr_llink1.002 -> fr_link1
- joint fr_joint3: child fr_llink3.002 -> fr_link3; origin xyz=-0.05995 -0.08004 -0.00055 rpy=0.00000 0.00000 0.00000 -> xyz=-0.05995 -0.08004 -0.00055 rpy=0.00000 0.00000 -0.00000; parent fr_llink2.002 -> fr_link2
- joint fr_joint4: child fr_llink4.002 -> fr_link4; origin xyz=-0.10341 0.07891 0.00044 rpy=0.00000 0.00000 0.00000 -> xyz=-0.10341 0.07891 0.00044 rpy=0.00000 0.00000 -0.00000; parent fr_llink3.002 -> fr_link3
