Commit message: Update mesh

File: quadson_bullet/assets/urdf/quadson.urdf (robot description, URDF)
Before this commit: robot quadson, 21 links, 21 joints
Joints:
- removed joint fl_jjoint1
- removed joint fl_joint5
- added joint fl_joint1: type revolute, parent fl_link0, child fl_link1, origin xyz=-0.00040 0.01862 0.05430 rpy=-1.57080 1.57080 -0.00000, axis 0.00000 0.00000 1.00000, limit lower=-3.14000 upper=3.14000 effort=0.00000 velocity=0.00000
