Commit message: Fix the warning of lacking inertia

File: quadson_sim/assets/whole_body/urdf/quadson_modified.urdf (robot description, URDF)
Before this commit: robot quadson, 25 links, 24 joints
Links:
- link fl_link4_dummy: mass None -> 0.0001
- link fr_link4_dummy: mass None -> 0.0001
- link rl_link4_dummy: mass None -> 0.0001
- link rr_link4_dummy: mass None -> 0.0001
