Commit message: Enable slider control whole body joint

File: quadson_sim/assets/whole_body/urdf/quadson.urdf (robot description, URDF)
Before this commit: robot quadson, 25 links, 24 joints
Links:
- removed link fl_link3
- removed link fl_link4_dummy
- removed link fr_link3
- removed link fr_link4_dummy
- removed link rl_link3
- removed link rl_link4_dummy
- removed link rr_link3
- removed link rr_link4_dummy
- added link fl_link5, mass 0.30000; visual mesh filename=../meshes/stl/fl_link5.stl scale=1.00000 1.00000 1.00000
- added link fr_link5, mass 0.30000; visual mesh filename=../meshes/stl/fr_link5.stl scale=1.00000 1.00000 1.00000
- added link rl_link5, mass 0.30000; visual mesh filename=../meshes/stl/rl_link5.stl scale=1.00000 1.00000 1.00000
- added link rr_link5, mass 0.30000; visual mesh filename=../meshes/stl/rr_link5.stl scale=1.00000 1.00000 1.00000
- link fl_link0: mass 0.30000 -> 0.50000
- link fl_link1: mass 0.10000 -> 0.30000
- link fl_link2: mass 0.10000 -> 0.30000
- link fl_link4: mass 0.10000 -> 0.30000
- link fr_link0: mass 0.30000 -> 0.50000
- link fr_link1: mass 0.10000 -> 0.30000
- link fr_link2: mass 0.10000 -> 0.30000
- link fr_link4: mass 0.10000 -> 0.30000; geometry visual mesh filename=../meshes/stl/fr_link4.001.stl scale=1.00000 1.00000 1.00000
- link rl_link0: mass 0.30000 -> 0.50000
- link rl_link1: mass 0.10000 -> 0.30000
- link rl_link2: mass 0.10000 -> 0.30000
- link rl_link4: mass 0.10000 -> 0.30000
- link rr_link0: mass 0.30000 -> 0.50000
- link rr_link1: mass 0.10000 -> 0.30000
- link rr_link2: mass 0.10000 -> 0.30000
- link rr_link4: mass 0.10000 -> 0.30000
Joints:
- removed joint fl_joint3
- removed joint fr_joint3
- removed joint rl_joint3
- removed joint rr_joint3
- joint fl_joint0: origin xyz=0.20500 0.09541 0.00215 rpy=0.00000 1.57080 0.00000 -> xyz=0.20500 0.09541 0.00215 rpy=-0.00000 1.57080 0.00000
- joint fl_joint4: origin xyz=-0.12919 -0.01447 0.00000 rpy=-0.00000 0.00000 0.00000 -> xyz=-0.00001 0.07999 0.00825 rpy=-0.00000 0.00000 0.00000; parent fl_link3 -> fl_link5
- joint fl_joint5: child fl_link4_dummy -> fl_link5
- joint fr_joint0: origin xyz=0.20500 -0.09380 0.00162 rpy=0.00000 1.57080 0.00000 -> xyz=0.20500 -0.09380 0.00162 rpy=-0.00000 1.57080 0.00000
- joint fr_joint1: origin xyz=-0.00026 -0.01767 -0.05190 rpy=1.01743 1.57079 2.58823 -> xyz=-0.00026 -0.01767 -0.05190 rpy=-1.57080 -1.57080 0.00000
- joint fr_joint2: origin xyz=-0.07999 -0.00001 -0.00825 rpy=-0.00000 0.00000 0.00000 -> xyz=0.07999 0.00001 -0.00825 rpy=-0.00000 0.00000 0.00000
- joint fr_joint4: origin xyz=0.12919 0.01447 -0.00000 rpy=0.00000 0.00000 -0.00000 -> xyz=-0.00001 0.07999 -0.00825 rpy=-0.00000 0.00000 0.00000; parent fr_link3 -> fr_link5
- joint fr_joint5: child fr_link4_dummy -> fr_link5; origin xyz=-0.00023 -0.01767 -0.13390 rpy=1.01743 1.57079 2.58823 -> xyz=-0.00023 -0.01767 -0.13390 rpy=-1.57080 -1.57080 0.00000
- joint rl_joint0: origin xyz=-0.20500 0.09541 0.00215 rpy=-3.14159 1.57080 0.00000 -> xyz=-0.20500 0.09541 0.00215 rpy=0.00000 -1.57080 0.00000
- joint rl_joint1: origin xyz=-0.00026 -0.01767 -0.05190 rpy=-2.50547 1.57080 -0.93467 -> xyz=0.00026 0.01767 -0.05190 rpy=1.57080 1.57080 0.00000
- joint rl_joint2: origin xyz=-0.07999 -0.00001 -0.00825 rpy=0.00000 -0.00000 -0.00000 -> xyz=-0.07999 -0.00001 -0.00825 rpy=0.00000 0.00000 -0.00000
- joint rl_joint4: origin xyz=0.12919 0.01447 -0.00000 rpy=0.00000 -0.00000 -0.00000 -> xyz=0.00001 -0.07999 -0.00825 rpy=0.00000 0.00000 0.00000; parent rl_link3 -> rl_link5
- joint rl_joint5: child rl_link4_dummy -> rl_link5; origin xyz=-0.00023 -0.01767 -0.13390 rpy=-2.50547 1.57080 -0.93467 -> xyz=0.00023 0.01767 -0.13390 rpy=1.57080 1.57080 0.00000
- joint rr_joint0: origin xyz=-0.20500 -0.09459 0.00215 rpy=-3.14159 1.57080 -0.00000 -> xyz=-0.20500 -0.09459 0.00215 rpy=0.00000 -1.57080 0.00000
- joint rr_joint1: origin xyz=-0.00011 0.01748 -0.05170 rpy=1.57080 -1.57080 -3.14159 -> xyz=0.00011 -0.01748 -0.05170 rpy=1.57080 1.57080 0.00000
- joint rr_joint2: origin xyz=0.07999 0.00001 0.00825 rpy=-0.00000 -0.00000 -0.00000 -> xyz=-0.07999 -0.00001 0.00825 rpy=0.00000 0.00000 -0.00000
- joint rr_joint4: origin xyz=-0.12919 -0.01447 0.00000 rpy=-0.00000 0.00000 -0.00000 -> xyz=0.00001 -0.07999 0.00825 rpy=0.00000 0.00000 -0.00000; parent rr_link3 -> rr_link5
- joint rr_joint5: child rr_link4_dummy -> rr_link5; origin xyz=-0.00008 0.01748 -0.13370 rpy=1.57080 -1.57080 -3.14159 -> xyz=0.00008 -0.01748 -0.13370 rpy=1.57080 1.57080 0.00000

File: quadson_sim/assets/whole_body/urdf/quadson_modified.urdf (robot description, URDF)
Before this commit: robot quadson, 25 links, 24 joints
Links:
- removed link fl_link3
- removed link fl_link4_dummy
- removed link fr_link3
- removed link fr_link4_dummy
- removed link rl_link3
- removed link rl_link4_dummy
- removed link rr_link3
- removed link rr_link4_dummy
- added link fl_link5, mass 0.30000; collision mesh filename=../meshes/stl/fl_link5.stl scale=1.00000 1.00000 1.00000; visual mesh filename=../meshes/stl/fl_link5.stl scale=1.00000 1.00000 1.00000
- added link fr_link5, mass 0.30000; collision mesh filename=../meshes/stl/fr_link5.stl scale=1.00000 1.00000 1.00000; visual mesh filename=../meshes/stl/fr_link5.stl scale=1.00000 1.00000 1.00000
- added link rl_link5, mass 0.30000; collision mesh filename=../meshes/stl/rl_link5.stl scale=1.00000 1.00000 1.00000; visual mesh filename=../meshes/stl/rl_link5.stl scale=1.00000 1.00000 1.00000
- added link rr_link5, mass 0.30000; collision mesh filename=../meshes/stl/rr_link5.stl scale=1.00000 1.00000 1.00000; visual mesh filename=../meshes/stl/rr_link5.stl scale=1.00000 1.00000 1.00000
- link fl_link0: mass 0.30000 -> 0.50000
- link fl_link1: mass 0.10000 -> 0.30000
- link fl_link2: mass 0.10000 -> 0.30000
- link fl_link4: mass 0.10000 -> 0.30000
- link fr_link0: mass 0.30000 -> 0.50000
- link fr_link1: mass 0.10000 -> 0.30000
- link fr_link2: mass 0.10000 -> 0.30000
- link fr_link4: mass 0.10000 -> 0.30000; geometry collision mesh filename=../meshes/stl/fr_link4.001.stl scale=1.00000 1.00000 1.00000; visual mesh filename=../meshes/stl/fr_link4.001.stl scale=1.00000 1.00000 1.00000
- link rl_link0: mass 0.30000 -> 0.50000
- link rl_link1: mass 0.10000 -> 0.30000
- link rl_link2: mass 0.10000 -> 0.30000
- link rl_link4: mass 0.10000 -> 0.30000
- link rr_link0: mass 0.30000 -> 0.50000
- link rr_link1: mass 0.10000 -> 0.30000
- link rr_link2: mass 0.10000 -> 0.30000
- link rr_link4: mass 0.10000 -> 0.30000
Joints:
- removed joint fl_joint3
- removed joint fr_joint3
- removed joint rl_joint3
- removed joint rr_joint3
- joint fl_joint0: origin xyz=0.20500 0.09541 0.00215 rpy=0.00000 1.57080 0.00000 -> xyz=0.20500 0.09541 0.00215 rpy=-0.00000 1.57080 0.00000
- joint fl_joint4: origin xyz=-0.12919 -0.01447 0.00000 rpy=-0.00000 0.00000 0.00000 -> xyz=-0.00001 0.07999 0.00825 rpy=-0.00000 0.00000 0.00000; parent fl_link3 -> fl_link5
- joint fl_joint5: child fl_link4_dummy -> fl_link5
- joint fr_joint0: origin xyz=0.20500 -0.09380 0.00162 rpy=0.00000 1.57080 0.00000 -> xyz=0.20500 -0.09380 0.00162 rpy=-0.00000 1.57080 0.00000
- joint fr_joint1: origin xyz=-0.00026 -0.01767 -0.05190 rpy=1.01743 1.57079 2.58823 -> xyz=-0.00026 -0.01767 -0.05190 rpy=-1.57080 -1.57080 0.00000
- joint fr_joint2: origin xyz=-0.07999 -0.00001 -0.00825 rpy=-0.00000 0.00000 0.00000 -> xyz=0.07999 0.00001 -0.00825 rpy=-0.00000 0.00000 0.00000
- joint fr_joint4: origin xyz=0.12919 0.01447 -0.00000 rpy=0.00000 0.00000 -0.00000 -> xyz=-0.00001 0.07999 -0.00825 rpy=-0.00000 0.00000 0.00000; parent fr_link3 -> fr_link5
- joint fr_joint5: child fr_link4_dummy -> fr_link5; origin xyz=-0.00023 -0.01767 -0.13390 rpy=1.01743 1.57079 2.58823 -> xyz=-0.00023 -0.01767 -0.13390 rpy=-1.57080 -1.57080 0.00000
- joint rl_joint0: origin xyz=-0.20500 0.09541 0.00215 rpy=-3.14159 1.57080 0.00000 -> xyz=-0.20500 0.09541 0.00215 rpy=0.00000 -1.57080 0.00000
- joint rl_joint1: origin xyz=-0.00026 -0.01767 -0.05190 rpy=-2.50547 1.57080 -0.93467 -> xyz=0.00026 0.01767 -0.05190 rpy=1.57080 1.57080 0.00000
- joint rl_joint2: origin xyz=-0.07999 -0.00001 -0.00825 rpy=0.00000 -0.00000 -0.00000 -> xyz=-0.07999 -0.00001 -0.00825 rpy=0.00000 0.00000 -0.00000
- joint rl_joint4: origin xyz=0.12919 0.01447 -0.00000 rpy=0.00000 -0.00000 -0.00000 -> xyz=0.00001 -0.07999 -0.00825 rpy=0.00000 0.00000 0.00000; parent rl_link3 -> rl_link5
- joint rl_joint5: child rl_link4_dummy -> rl_link5; origin xyz=-0.00023 -0.01767 -0.13390 rpy=-2.50547 1.57080 -0.93467 -> xyz=0.00023 0.01767 -0.13390 rpy=1.57080 1.57080 0.00000
- joint rr_joint0: origin xyz=-0.20500 -0.09459 0.00215 rpy=-3.14159 1.57080 -0.00000 -> xyz=-0.20500 -0.09459 0.00215 rpy=0.00000 -1.57080 0.00000
- joint rr_joint1: origin xyz=-0.00011 0.01748 -0.05170 rpy=1.57080 -1.57080 -3.14159 -> xyz=0.00011 -0.01748 -0.05170 rpy=1.57080 1.57080 0.00000
- joint rr_joint2: origin xyz=0.07999 0.00001 0.00825 rpy=-0.00000 -0.00000 -0.00000 -> xyz=-0.07999 -0.00001 0.00825 rpy=0.00000 0.00000 -0.00000
- joint rr_joint4: origin xyz=-0.12919 -0.01447 0.00000 rpy=-0.00000 0.00000 -0.00000 -> xyz=0.00001 -0.07999 0.00825 rpy=0.00000 0.00000 -0.00000; parent rr_link3 -> rr_link5
- joint rr_joint5: child rr_link4_dummy -> rr_link5; origin xyz=-0.00008 0.01748 -0.13370 rpy=1.57080 -1.57080 -3.14159 -> xyz=0.00008 -0.01748 -0.13370 rpy=1.57080 1.57080 0.00000
