Commit message: Update single leg, achieve closed chain

File: quadson_sim/assets/single_leg/urdf/single_leg.urdf (robot description, URDF)
Before this commit: robot single_leg, 6 links, 5 joints
Links:
- removed link link0_link
- removed link link1_link
- removed link link2_link
- removed link link3_link
- removed link link4_dummy_link
- removed link link4_link
- added link link0, mass 0.20000; visual mesh filename=../meshes/stl/link0.stl scale=1.00000 1.00000 1.00000
- added link link1, mass 0.20000; visual mesh filename=../meshes/stl/link1.stl scale=1.00000 1.00000 1.00000
- added link link2, mass 0.20000; visual mesh filename=../meshes/stl/link2.stl scale=1.00000 1.00000 1.00000
- added link link3, mass 0.20000; visual mesh filename=../meshes/stl/link3.stl scale=1.00000 1.00000 1.00000
- added link link4, mass 0.20000; visual mesh filename=../meshes/stl/link4.stl scale=1.00000 1.00000 1.00000
Joints:
- removed joint joint3
- joint joint1: child link1_link -> link1; origin xyz=0.04100 0.01800 -0.00000 rpy=-1.57080 0.00000 0.00000 -> xyz=0.04100 0.01800 0.00003 rpy=-1.57080 0.00000 0.00000; parent link0_link -> link0
- joint joint2: child link2_link -> link2; origin xyz=0.00001 0.07999 0.00825 rpy=-0.00000 0.00000 0.00000 -> xyz=0.07999 0.00001 0.00825 rpy=-0.00000 0.00000 0.00000; parent link1_link -> link1
- joint joint4: child link4_link -> link3; origin xyz=-0.03281 -0.09447 -0.00000 rpy=-0.00000 0.00000 0.00000 -> xyz=-0.00001 0.07999 0.00825 rpy=-0.00000 0.00000 0.00000; parent link3_link -> link4
- joint joint5: child link4_dummy_link -> link4; origin xyz=-0.04100 0.01800 0.00003 rpy=-1.57080 0.00000 0.00000 -> xyz=-0.04100 0.01800 -0.00000 rpy=-1.57080 0.00000 0.00000; parent link0_link -> link0

File: quadson_sim/assets/single_leg/urdf/single_leg_modified.urdf (robot description, URDF)
Before this commit: robot single_leg, 6 links, 5 joints
Links:
- removed link link0_link
- removed link link1_link
- removed link link2_link
- removed link link3_link
- removed link link4_dummy_link
- removed link link4_link
- added link link0, mass 0.20000; collision mesh filename=../meshes/stl/link0.stl scale=1.00000 1.00000 1.00000; visual mesh filename=../meshes/stl/link0.stl scale=1.00000 1.00000 1.00000
- added link link1, mass 0.20000; collision mesh filename=../meshes/stl/link1.stl scale=1.00000 1.00000 1.00000; visual mesh filename=../meshes/stl/link1.stl scale=1.00000 1.00000 1.00000
- added link link2, mass 0.20000; collision mesh filename=../meshes/stl/link2.stl scale=1.00000 1.00000 1.00000; visual mesh filename=../meshes/stl/link2.stl scale=1.00000 1.00000 1.00000
- added link link3, mass 0.20000; collision mesh filename=../meshes/stl/link3.stl scale=1.00000 1.00000 1.00000; visual mesh filename=../meshes/stl/link3.stl scale=1.00000 1.00000 1.00000
- added link link4, mass 0.20000; collision mesh filename=../meshes/stl/link4.stl scale=1.00000 1.00000 1.00000; visual mesh filename=../meshes/stl/link4.stl scale=1.00000 1.00000 1.00000
Joints:
- removed joint joint3
- joint joint1: child link1_link -> link1; origin xyz=0.04100 0.01800 -0.00000 rpy=-1.57080 0.00000 0.00000 -> xyz=0.04100 0.01800 0.00003 rpy=-1.57080 0.00000 0.00000; parent link0_link -> link0
- joint joint2: child link2_link -> link2; origin xyz=0.00001 0.07999 0.00825 rpy=-0.00000 0.00000 0.00000 -> xyz=0.07999 0.00001 0.00825 rpy=-0.00000 0.00000 0.00000; parent link1_link -> link1
- joint joint4: child link4_link -> link3; origin xyz=-0.03281 -0.09447 -0.00000 rpy=-0.00000 0.00000 0.00000 -> xyz=-0.00001 0.07999 0.00825 rpy=-0.00000 0.00000 0.00000; parent link3_link -> link4
- joint joint5: child link4_dummy_link -> link4; origin xyz=-0.04100 0.01800 0.00003 rpy=-1.57080 0.00000 0.00000 -> xyz=-0.04100 0.01800 -0.00000 rpy=-1.57080 0.00000 0.00000; parent link0_link -> link0
